File: pcb/CopperPilotDrone.kicad_pcb (KiCad board)
At the start: 2 copper layers, 100 x 100 mm, 140 parts, among them IC1 TP4056, J1 USB_C_Receptacle_USB2.0, J2 Conn_01x02_Female, J3 B2B-PH-SM4-TB(LF)(SN), J4 Conn_01x02_Female, J5 Conn_01x02_Female, J6 Conn_01x02_Female, SW1 PCM12SMTR, SW2 TS-1187A, SW3 TS-1187A, T1 SI2302DS-T1, T2 SI2302DS-T1, T3 SI2302DS-T1, T4 SI2302DS-T1, U2 AO3401, U3 AP2112K-3.3TRG1, U8 ESP32-S3-WROOM-1-N8R8, U9 MPU-6050

Commit message: fix(dfm): resolve via-to-pad, slot width, annular ring, and acute corner DFM issues
Reposition 7 vias away from adjacent SMD pads, widen J1 USB-C shield slots from 0.60mm to 0.85mm, upgrade 0.35mm drill vias from 0.65mm to 0.68mm pad diameter (0.165mm annular ring), chamfer acute bends on +3V3 and /D+, and increase +3V3 trace-to-mask clearance near U3.

Co-Authored-By: CopperPilot <noreply@copperpilot.ai>
Routing:
- net +3V3: track 86.3 -> 84.7 mm
- net Net-(C15-Pad2): track 1.21 -> 2.04 mm
